Commit message: Adding camera to wrist of robot, fixed joint

File: src/ur10_description/urdf/ur10.urdf.xacro (robot description, xacro)
@@ -271,4 +271,44 @@
       </collision>
     </link>
+    <link name="${prefix}camera_link">
+		<!--<pose> 0 0 0 0 0 0 </pose> !-->
+		<inertial>
+		    <origin xyz="0.0 0.0 0.05" rpy="0 0 0"/>
+		    <mass value="1"/>
+		    <inertia
+			ixx="1.0" ixy="0.0" ixz="0.0"
+			iyy="1.0" iyz="0.0"
+			izz="1.0"/>
+	    	</inertial>
+		<collision name="collisionBox">
+		    	<origin xyz="0.0 0.0 0.0" rpy="0 0 0"/>
+			<geometry>
+			<box size="0.1 0.03 0.05"/>
+			</geometry>
+		</collision>
+		<visual name="visualBox">
+		    	<origin xyz="0.0 0.0 0.0" rpy="0 0 0"/>
+			<geometry>
+			<box size="0.1 0.03 0.05"/>
+			</geometry>
+		</visual>
+		<collision name="collisionLense">
+			<origin xyz="0.0 0.02 0.01" rpy="1.5707963 0 0" />
+			<geometry>
+				<cylinder length="0.02" radius="0.02"/>
+			</geometry>
+		</collision>
+		<visual name="visualLense">
+			<origin xyz="0.0 0.02 0.01" rpy="1.5707963 0 0" />
+			<geometry>
+				<cylinder length="0.02" radius="0.02"/>
+			</geometry>
+		</visual>
+	</link>
+    <joint name="${prefix}camera_joint" type="fixed">
+      <parent link="${prefix}wrist_1_link" />
+      <child link = "${prefix}camera_link" />
+      <origin xyz="-0.08 ${wrist_3_length} ${wrist_1_length}" rpy="0.0 0.0 ${pi/2.0}" />
+    </joint>
     <xacro:ur10_arm_transmission prefix="${prefix}" />
     <xacro:ur10_arm_gazebo prefix="${prefix}" />

File: src/ur10_description/urdf/ur10_robot.urdf (robot description, URDF)
Before this commit: robot ur10, 9 links, 8 joints
Links:
- added link base
- added link camera_link, mass 1; collision box size=0.1 0.03 0.05; collision cylinder length=0.02 radius=0.02
- added link tool0
Joints:
- added joint base_link-base_fixed_joint: type fixed, parent base_link, child base, origin xyz=0 0 0 rpy=0 0 -3.14159265
- added joint camera_joint: type fixed, parent wrist_1_link, child camera_link, origin xyz=-0.08 0.0922 0.1149 rpy=0.0 0.0 1.570796325
- added joint wrist_3_link-tool0_fixed_joint: type fixed, parent wrist_3_link, child tool0, origin xyz=0 0.0922 0 rpy=-1.570796325 0 0

Commit message: making gazebo camera xacro

File: src/ur10_description/urdf/ur10.urdf.xacro (robot description, xacro)
@@ -309,6 +309,41 @@
       <parent link="${prefix}wrist_1_link" />
       <child link = "${prefix}camera_link" />
-      <origin xyz="-0.08 ${wrist_3_length} ${wrist_1_length}" rpy="0.0 0.0 ${pi/2.0}" />
-    </joint>
+      <origin xyz="-0.08 ${wrist_3_length} 0" rpy="0.0 0.0 ${pi/2.0}" />
+    </joint>
+	<gazebo reference = "${prefix}camera_link">
+		<sensor  type="camera" name="Camera Sensor">
+        		<origin xyz="0 0 0" rpy="0 0 0" />
+			<update_rate>50</update_rate>
+			<always_on>true</always_on>
+			<visualize>true</visualize>
+			<camera>
+				<horizontal_fov>1.047</horizontal_fov>
+				<image>
+					<height>786</height>
+					<width>786</width>
+				</image>
+				<!--<save enabled=True>
+					<path>"~/CameraData"</path>
+				</save>-->
+				<noise>
+				    <type>gaussian</type>
+				    <mean>0.0</mean>
+				    <stddev>0.01</stddev>
+				</noise>
+				<clip>
+				    <near>0.1</near>
+				    <far>100</far>
+				</clip>
+				<distortion>
+				   <k1>-0.25</k1>
+				   <k2>0.12</k2>
+				   <k3>0.0</k3>
+				   <p1>-0.00028</p1>
+				   <p2>-0.00005</p2>
+				   <center>0.5 0.5</center>
+				</distortion>
+			</camera>
+		</sensor>
+	</gazebo>
     <xacro:ur10_arm_transmission prefix="${prefix}" />
     <xacro:ur10_arm_gazebo prefix="${prefix}" />

File: src/ur10_description/urdf/ur10_robot.urdf (robot description, URDF)
Before this commit: robot ur10, 12 links, 11 joints
Joints:
- joint camera_joint: origin xyz=-0.08 0.0922 0.1149 rpy=0.0 0.0 1.570796325 -> xyz=-0.08 0.0922 0 rpy=0.0 0.0 1.570796325

Commit message: adding camera plugin

File: src/ur10_description/urdf/ur10.urdf.xacro (robot description, xacro)
@@ -309,13 +309,13 @@
       <parent link="${prefix}wrist_1_link" />
       <child link = "${prefix}camera_link" />
-      <origin xyz="-0.08 ${wrist_3_length} 0" rpy="0.0 0.0 ${pi/2.0}" />
+      <origin xyz="-0.06 ${wrist_3_length} 0" rpy="0.0 0.0 ${pi/2.0}" />
     </joint>
 	<gazebo reference = "${prefix}camera_link">
 		<sensor  type="camera" name="Camera Sensor">
-        		<origin xyz="0 0 0" rpy="0 0 0" />
 			<update_rate>50</update_rate>
 			<always_on>true</always_on>
 			<visualize>true</visualize>
 			<camera>
+				<pose> 0.0 0.0 0.0 0.0 0.0 0.0</pose>
 				<horizontal_fov>1.047</horizontal_fov>
 				<image>
@@ -344,4 +344,18 @@
 				</distortion>
 			</camera>
+		        <plugin name="camera_controller" filename="libgazebo_ros_camera.so">
+		            <alwaysOn>true</alwaysOn>
+		            <updateRate>0.0</updateRate>
+		            <cameraName>Arm/camera</cameraName>
+		            <imageTopicName>image_raw</imageTopicName>
+		            <cameraInfoTopicName>camera_info</cameraInfoTopicName>
+		            <frameName>${prefix}camera_link</frameName>
+		            <hackBaseline>0.07</hackBaseline>
+		            <distortionK1>0.0</distortionK1>
+		            <distortionK2>0.0</distortionK2>
+		            <distortionK3>0.0</distortionK3>
+		            <distortionT1>0.0</distortionT1>
+		            <distortionT2>0.0</distortionT2>
+		        </plugin>
 		</sensor>
 	</gazebo>

File: src/ur10_description/urdf/ur10_robot.urdf (robot description, URDF)
Before this commit: robot ur10, 12 links, 11 joints
Joints:
- joint base_link-base_fixed_joint: origin xyz=0 0 0 rpy=0 0 -3.14159265 -> xyz=0 0 0 rpy=0 0 -3.14159265359
- joint camera_joint: origin xyz=-0.08 0.0922 0 rpy=0.0 0.0 1.570796325 -> xyz=-0.06 0.0922 0 rpy=0.0 0.0 1.57079632679
- joint ee_fixed_joint: origin xyz=0.0 0.0922 0.0 rpy=0.0 0.0 1.570796325 -> xyz=0.0 0.0922 0.0 rpy=0.0 0.0 1.57079632679
- joint elbow_joint: limit lower=-6.2831853 upper=6.2831853 effort=150.0 velocity=3.15 -> lower=-6.28318530718 upper=6.28318530718 effort=150.0 velocity=3.15
- joint shoulder_lift_joint: limit lower=-6.2831853 upper=6.2831853 effort=330.0 velocity=2.16 -> lower=-6.28318530718 upper=6.28318530718 effort=330.0 velocity=2.16; origin xyz=0.0 0.220941 0.0 rpy=0.0 1.570796325 0.0 -> xyz=0.0 0.220941 0.0 rpy=0.0 1.57079632679 0.0
- joint shoulder_pan_joint: limit lower=-6.2831853 upper=6.2831853 effort=330.0 velocity=2.16 -> lower=-6.28318530718 upper=6.28318530718 effort=330.0 velocity=2.16
- joint wrist_1_joint: limit lower=-6.2831853 upper=6.2831853 effort=54.0 velocity=3.2 -> lower=-6.28318530718 upper=6.28318530718 effort=54.0 velocity=3.2; origin xyz=0.0 0.0 0.5723 rpy=0.0 1.570796325 0.0 -> xyz=0.0 0.0 0.5723 rpy=0.0 1.57079632679 0.0
- joint wrist_2_joint: limit lower=-6.2831853 upper=6.2831853 effort=54.0 velocity=3.2 -> lower=-6.28318530718 upper=6.28318530718 effort=54.0 velocity=3.2
- joint wrist_3_joint: limit lower=-6.2831853 upper=6.2831853 effort=54.0 velocity=3.2 -> lower=-6.28318530718 upper=6.28318530718 effort=54.0 velocity=3.2
- joint wrist_3_link-tool0_fixed_joint: origin xyz=0 0.0922 0 rpy=-1.570796325 0 0 -> xyz=0 0.0922 0 rpy=-1.57079632679 0 0

Commit message: Fixing camera pose, shrinking camera, adding a second  camera, changing camera joint

File: src/ur10_description/urdf/ur10.urdf.xacro (robot description, xacro)
@@ -271,5 +271,5 @@
       </collision>
     </link>
-    <link name="${prefix}camera_link">
+    <link name="${prefix}down_camera_link">
 		<!--<pose> 0 0 0 0 0 0 </pose> !-->
 		<inertial>
@@ -284,5 +284,5 @@
 		    	<origin xyz="0.0 0.0 0.0" rpy="0 0 0"/>
 			<geometry>
-			<box size="0.1 0.03 0.05"/>
+			<box size="0.03 0.03 0.03"/>
 			</geometry>
 		</collision>
@@ -290,9 +290,10 @@
 		    	<origin xyz="0.0 0.0 0.0" rpy="0 0 0"/>
 			<geometry>
-			<box size="0.1 0.03 0.05"/>
+			<box size="0.03 0.03 0.03"/>
 			</geometry>
 		</visual>
+		<!--   The circular lense if commented out due to the diffuculty of tuning/finding the right rpy configurations
 		<collision name="collisionLense">
-			<origin xyz="0.0 0.02 0.01" rpy="1.5707963 0 0" />
+			<origin xyz="0.0 0.0 -0.02" rpy="0 ${pi/2.0} 0"/>
 			<geometry>
 				<cylinder length="0.02" radius="0.02"/>
@@ -300,17 +301,17 @@
 		</collision>
 		<visual name="visualLense">
-			<origin xyz="0.0 0.02 0.01" rpy="1.5707963 0 0" />
+			<origin xyz="0.0 0.0 -0.02" rpy="0 ${pi/2.0} 0"/>
 			<geometry>
 				<cylinder length="0.02" radius="0.02"/>
 			</geometry>
-		</visual>
+		</visual> !-->
 	</link>
-    <joint name="${prefix}camera_joint" type="fixed">
-      <parent link="${prefix}wrist_1_link" />
-      <child link = "${prefix}camera_link" />
-      <origin xyz="-0.06 ${wrist_3_length} 0" rpy="0.0 0.0 ${pi/2.0}" />
-    </joint>
-	<gazebo reference = "${prefix}camera_link">
-		<sensor  type="camera" name="Camera Sensor">
+    <joint name="${prefix}down_camera_joint" type="fixed">
+      <parent link="${prefix}wrist_2_link" />
+      <child link = "${prefix}down_camera_link" />
+      <origin xyz="-0.06 0.0 0.12" rpy="0.0 ${-pi/2.0} ${pi/2.0}" />
+    </joint>
+    <gazebo reference = "${prefix}down_camera_link">
+		<sensor  type="camera" name="Down Camera Sensor">
 			<update_rate>50</update_rate>
 			<always_on>true</always_on>
@@ -344,11 +345,101 @@
 				</distortion>
 			</camera>
-		        <plugin name="camera_controller" filename="libgazebo_ros_camera.so">
+		        <plugin name="down_camera_controller" filename="libgazebo_ros_camera.so">
 		            <alwaysOn>true</alwaysOn>
 		            <updateRate>0.0</updateRate>
-		            <cameraName>Arm/camera</cameraName>
+		            <cameraName>Arm/down_camera</cameraName>
 		            <imageTopicName>image_raw</imageTopicName>
 		            <cameraInfoTopicName>camera_info</cameraInfoTopicName>
-		            <frameName>${prefix}camera_link</frameName>
+		            <frameName>${prefix}down_camera_link</frameName>
+		            <hackBaseline>0.07</hackBaseline>
+		            <distortionK1>0.0</distortionK1>
+		            <distortionK2>0.0</distortionK2>
+		            <distortionK3>0.0</distortionK3>
+		            <distortionT1>0.0</distortionT1>
+		            <distortionT2>0.0</distortionT2>
+		        </plugin>
+		</sensor>
+	</gazebo>
+	<link name="${prefix}right_camera_link">
+		<!--<pose> 0 0 0 0 0 0 </pose> !-->
+		<inertial>
+		    <origin xyz="0.0 0.0 0.05" rpy="0 0 0"/>
+		    <mass value="1"/>
+		    <inertia
+			ixx="1.0" ixy="0.0" ixz="0.0"
+			iyy="1.0" iyz="0.0"
+			izz="1.0"/>
+	    	</inertial>
+		<collision name="collisionBox">
+		    	<origin xyz="0.0 0.0 0.0" rpy="0 0 0"/>
+			<geometry>
+			<box size="0.03 0.03 0.03"/>
+			</geometry>
+		</collision>
+		<visual name="visualBox">
+		    	<origin xyz="0.0 0.0 0.0" rpy="0 0 0"/>
+			<geometry>
+			<box size="0.03 0.03 0.03"/>
+			</geometry>
+		</visual>
+		<!--   The circular lense if commented out due to the diffuculty of tuning/finding the right rpy configurations
+		<collision name="collisionLense">
+			<origin xyz="0.0 0.0 -0.02" rpy="0 ${pi/2.0} 0"/>
+			<geometry>
+				<cylinder length="0.02" radius="0.02"/>
+			</geometry>
+		</collision>
+		<visual name="visualLense">
+			<origin xyz="0.0 0.0 -0.02" rpy="0 ${pi/2.0} 0"/>
+			<geometry>
+				<cylinder length="0.02" radius="0.02"/>
+			</geometry>
+		</visual> !-->
+	</link>
+    <joint name="${prefix}right_camera_joint" type="fixed">
+      <parent link="${prefix}wrist_2_link" />
+      <child link = "${prefix}right_camera_link" />
+      <origin xyz="-0.06 0.0 0.08" rpy="0.0 0.0 ${pi/2.0}" />
+    </joint>
+    <gazebo reference = "${prefix}right_camera_link">
+		<sensor  type="camera" name="Right Camera Sensor">
+			<update_rate>50</update_rate>
+			<always_on>true</always_on>
+			<visualize>true</visualize>
+			<camera>
+				<pose> 0.0 0.0 0.0 0.0 0.0 0.0</pose>
+				<horizontal_fov>1.047</horizontal_fov>
+				<image>
+					<height>786</height>
+					<width>786</width>
+				</image>
+				<!--<save enabled=True>
+					<path>"~/CameraData"</path>
+				</save>-->
+				<noise>
+				    <type>gaussian</type>
+				    <mean>0.0</mean>
+				    <stddev>0.01</stddev>
+				</noise>
+				<clip>
+				    <near>0.1</near>
+				    <far>100</far>
+				</clip>
+				<distortion>
+				   <k1>-0.25</k1>
+				   <k2>0.12</k2>
+				   <k3>0.0</k3>
+				   <p1>-0.00028</p1>
+				   <p2>-0.00005</p2>
+				   <center>0.5 0.5</center>
+				</distortion>
+			</camera>
+		        <plugin name="right_camera_controller" filename="libgazebo_ros_camera.so">
+		            <alwaysOn>true</alwaysOn>
+		            <updateRate>0.0</updateRate>
+		            <cameraName>Arm/right_camera</cameraName>
+		            <imageTopicName>image_raw</imageTopicName>
+		            <cameraInfoTopicName>camera_info</cameraInfoTopicName>
+		            <frameName>${prefix}right_camera_link</frameName>
 		            <hackBaseline>0.07</hackBaseline>
 		            <distortionK1>0.0</distortionK1>

File: src/ur10_description/urdf/ur10_robot.urdf (robot description, URDF)
Before this commit: robot ur10, 12 links, 11 joints
Links:
- removed link camera_link
- added link down_camera_link, mass 1; collision box size=0.03 0.03 0.03; visual box size=0.03 0.03 0.03
- added link right_camera_link, mass 1; collision box size=0.03 0.03 0.03; visual box size=0.03 0.03 0.03
Joints:
- removed joint camera_joint
- added joint down_camera_joint: type fixed, parent wrist_2_link, child down_camera_link, origin xyz=-0.06 0.0 0.12 rpy=0.0 -1.57079632679 1.57079632679
- added joint right_camera_joint: type fixed, parent wrist_2_link, child right_camera_link, origin xyz=-0.06 0.0 0.08 rpy=0.0 0.0 1.57079632679

Commit message: Camera comments added

File: src/ur10_description/urdf/ur10.urdf.xacro (robot description, xacro)
@@ -271,6 +271,16 @@
       </collision>
     </link>
+<!-- Notes about camera in general
+* The gazebo tag is what actually makes the sensor, it is in SDF I beleive, not URDF
+* In order to change the sensor pose or even the link pose, use the pose fixed join associated with each camera
+* Recalculate the inertia statistics if you change the mass or shape of the camera
+* There are only 3 wrist links, we have attatched the cameras to the second
+* The cylindric camera lense has been removed, it was difficult to tune the pose (rpy)
+* Watch the frameName of the camera topics, they should match the link name
+* Tune the distortions to your needs
+* This code requires uncommenting if you want to save the images somewhere
+-->
+<!-- DOWN FACING CAMERA -->
     <link name="${prefix}down_camera_link">
-		<!--<pose> 0 0 0 0 0 0 </pose> !-->
 		<inertial>
 		    <origin xyz="0.0 0.0 0.05" rpy="0 0 0"/>
@@ -293,17 +303,4 @@
 			</geometry>
 		</visual>
-		<!--   The circular lense if commented out due to the diffuculty of tuning/finding the right rpy configurations
-		<collision name="collisionLense">
-			<origin xyz="0.0 0.0 -0.02" rpy="0 ${pi/2.0} 0"/>
-			<geometry>
-				<cylinder length="0.02" radius="0.02"/>
-			</geometry>
-		</collision>
-		<visual name="visualLense">
-			<origin xyz="0.0 0.0 -0.02" rpy="0 ${pi/2.0} 0"/>
-			<geometry>
-				<cylinder length="0.02" radius="0.02"/>
-			</geometry>
-		</visual> !-->
 	</link>
     <joint name="${prefix}down_camera_joint" type="fixed">
@@ -361,4 +358,5 @@
 		</sensor>
 	</gazebo>
+<!-- RIGHT FACING CAMERA -->
 	<link name="${prefix}right_camera_link">
 		<!--<pose> 0 0 0 0 0 0 </pose> !-->
@@ -383,17 +381,4 @@
 			</geometry>
 		</visual>
-		<!--   The circular lense if commented out due to the diffuculty of tuning/finding the right rpy configurations
-		<collision name="collisionLense">
-			<origin xyz="0.0 0.0 -0.02" rpy="0 ${pi/2.0} 0"/>
-			<geometry>
-				<cylinder length="0.02" radius="0.02"/>
-			</geometry>
-		</collision>
-		<visual name="visualLense">
-			<origin xyz="0.0 0.0 -0.02" rpy="0 ${pi/2.0} 0"/>
-			<geometry>
-				<cylinder length="0.02" radius="0.02"/>
-			</geometry>
-		</visual> !-->
 	</link>
     <joint name="${prefix}right_camera_joint" type="fixed">
@@ -451,4 +436,5 @@
 		</sensor>
 	</gazebo>
+<!-- END OF CODE ADDED-->
     <xacro:ur10_arm_transmission prefix="${prefix}" />
     <xacro:ur10_arm_gazebo prefix="${prefix}" />
