Commit message: Added gripper into robot.

File: src/ur_description/urdf/ur.gazebo.xacro (robot description, xacro)
@@ -23,4 +23,7 @@
       <selfCollide>true</selfCollide>
     </gazebo>
+    <gazebo reference="${prefix}gripper_link">
+      <selfCollide>true</selfCollide>
+    </gazebo>
   </xacro:macro>
 </robot>

File: src/ur_description/urdf/ur10.urdf.xacro (robot description, xacro)
@@ -34,4 +34,5 @@
     <xacro:property name="wrist_2_mass" value="1.96" />
     <xacro:property name="wrist_3_mass" value="0.202" />
+    <xacro:property name="gripper_mass" value="1.00" />
     <!-- These parameters are borrowed from the urcontrol.conf file
         but are not verified for the correct permutation.
@@ -316,4 +317,27 @@
       </collision>
     </link>
+    <joint name="${prefix}gripper_fixed_joint" type="fixed">
+      <parent link="${prefix}ee_link" />
+      <child link = "${prefix}gripper_link" />
+      <origin xyz="0.0 -0.05 0.1" rpy="0.0 ${pi/2.0} 0.0" />
+    </joint>
+    <link name="${prefix}gripper_link">
+      <visual>
+        <geometry>
+          <mesh filename="package://ur_description/meshes/ur10/visual/gripper.dae"/>
+        </geometry>
+        <material name="LightGrey">
+          <color rgba="0.7 0.7 0.7 1.0"/>
+        </material>
+      </visual>
+      <collision>
+        <geometry>
+          <mesh filename="package://ur_description/meshes/ur10/collision/gripper.stl"/>
+        </geometry>
+      </collision>
+      <xacro:cylinder_inertial radius="0.1" length="0.07" mass="${gripper_mass}">
+        <origin xyz="0.0 -0.05 0.1" rpy="0.0 ${pi/2.0} 0.0" />
+      </xacro:cylinder_inertial>
+    </link>
     <xacro:ur_arm_transmission prefix="${prefix}" hw_interface="${transmission_hw_interface}" />
     <xacro:ur_arm_gazebo prefix="${prefix}" />

Commit message: Fixed camera location.

File: src/ur_description/urdf/ur.gazebo.xacro (robot description, xacro)
@@ -26,4 +26,7 @@
       <selfCollide>true</selfCollide>
     </gazebo>
+    <!-- <gazebo reference="${prefix}depth_camera_link">
+      <selfCollide>true</selfCollide>
+    </gazebo> -->
   </xacro:macro>
 </robot>

File: src/ur_description/urdf/ur10.urdf.xacro (robot description, xacro)
@@ -288,7 +288,7 @@
     </link>
     <joint name="${prefix}depth_camera_joint" type="fixed">
-      <parent link="${prefix}wrist_2_link" />
+      <parent link="${prefix}gripper_link" />
       <child link = "${prefix}depth_camera_link" />
-      <origin xyz="-0.06 0.0 0.12" rpy="0.0 ${-pi/2.0} ${pi/2.0}" />
+      <origin xyz="0.0 -0.0151 0.0" rpy="0.0 0.0 0.0" />
     </joint>
     <gazebo reference = "${prefix}depth_camera_link">
