Commit message: Adding visual camera to ur10

File: src/ur_description/urdf/ur10.urdf.xacro (robot description, xacro)
@@ -266,4 +266,80 @@
       </xacro:cylinder_inertial>
     </link>
+    <link name="${prefix}depth_camera_link">
+    <inertial>
+        <origin xyz="0.0 0.0 0.05" rpy="0 0 0"/>
+        <mass value="1"/>
+        <inertia
+      ixx="1.0" ixy="0.0" ixz="0.0"
+      iyy="1.0" iyz="0.0"
+      izz="1.0"/>
+        </inertial>
+    <collision name="collisionBox">
+          <origin xyz="0.0 0.0 0.0" rpy="0 0 0"/>
+      <geometry>
+      <box size="0.03 0.03 0.03"/>
+      </geometry>
+    </collision>
+    <visual name="visualBox">
+          <origin xyz="0.0 0.0 0.0" rpy="0 0 0"/>
+      <geometry>
+      <box size="0.03 0.03 0.03"/>
+      </geometry>
+    </visual>
+  </link>
+    <joint name="${prefix}depth_camera_joint" type="fixed">
+      <parent link="${prefix}wrist_2_link" />
+      <child link = "${prefix}depth_camera_link" />
+      <origin xyz="-0.06 0.0 0.12" rpy="0.0 ${-pi/2.0} ${pi/2.0}" />
+    </joint>
+  <gazebo reference = "${prefix}depth_camera_link">
+    <sensor  type="camera" name="Depth Camera Sensor">
+      <update_rate>50</update_rate>
+      <always_on>true</always_on>
+      <visualize>true</visualize>
+      <camera>
+        <pose> 0.0 0.0 0.0 0.0 0.0 0.0</pose>
+        <horizontal_fov>1.047</horizontal_fov>
+        <image>
+          <height>786</height>
+          <width>786</width>
+        </image>
+        <!--<save enabled=True>
+          <path>"~/CameraData"</path>
+        </save>-->
+        <noise>
+            <type>gaussian</type>
+            <mean>0.0</mean>
+            <stddev>0.01</stddev>
+        </noise>
+        <clip>
+            <near>0.1</near>
+            <far>100</far>
+        </clip>
+        <distortion>
+           <k1>-0.25</k1>
+           <k2>0.12</k2>
+           <k3>0.0</k3>
+           <p1>-0.00028</p1>
+           <p2>-0.00005</p2>
+           <center>0.5 0.5</center>
+        </distortion>
+      </camera>
+            <plugin name="depth_camera_controller" filename="libgazebo_ros_camera.so">
+                <alwaysOn>true</alwaysOn>
+                <updateRate>0.0</updateRate>
+                <cameraName>Arm/depth_camera</cameraName>
+                <imageTopicName>image_raw</imageTopicName>
+                <cameraInfoTopicName>camera_info</cameraInfoTopicName>
+                <frameName>${prefix}depth_camera_link</frameName>
+                <hackBaseline>0.07</hackBaseline>
+                <distortionK1>0.0</distortionK1>
+                <distortionK2>0.0</distortionK2>
+                <distortionK3>0.0</distortionK3>
+                <distortionT1>0.0</distortionT1>
+                <distortionT2>0.0</distortionT2>
+            </plugin>
+    </sensor>
+  </gazebo>
     <joint name="${prefix}wrist_3_joint" type="revolute">
       <parent link="${prefix}wrist_2_link" />

Commit message: Formating changes.

File: src/ur_description/urdf/ur10.urdf.xacro (robot description, xacro)
@@ -272,21 +272,19 @@
         <mass value="1"/>
         <inertia
-      ixx="1.0" ixy="0.0" ixz="0.0"
-      iyy="1.0" iyz="0.0"
-      izz="1.0"/>
-        </inertial>
-    <collision name="collisionBox">
-          <origin xyz="0.0 0.0 0.0" rpy="0 0 0"/>
-      <geometry>
-      <box size="0.03 0.03 0.03"/>
-      </geometry>
-    </collision>
-    <visual name="visualBox">
-          <origin xyz="0.0 0.0 0.0" rpy="0 0 0"/>
-      <geometry>
-      <box size="0.03 0.03 0.03"/>
-      </geometry>
-    </visual>
-  </link>
+        ixx="1.0" ixy="0.0" ixz="0.0"
+        iyy="1.0" iyz="0.0"
+        izz="1.0"/>
+      </inertial>
+      <collision name="collisionBox">
+        <geometry>
+          <box size="0.03 0.03 0.03"/>
+        </geometry>
+      </collision>
+      <visual name="visualBox">
+        <geometry>
+          <box size="0.03 0.03 0.03"/>
+        </geometry>
+      </visual>
+    </link>
     <joint name="${prefix}depth_camera_joint" type="fixed">
       <parent link="${prefix}wrist_2_link" />
@@ -294,47 +292,47 @@
       <origin xyz="-0.06 0.0 0.12" rpy="0.0 ${-pi/2.0} ${pi/2.0}" />
     </joint>
-  <gazebo reference = "${prefix}depth_camera_link">
-    <sensor name="camera" type="depth">
-        <update_rate>20</update_rate>
-        <camera>
-          <horizontal_fov>1.047198</horizontal_fov>
-          <image>
-            <width>640</width>
-            <height>480</height>
-            <format>R8G8B8</format>
-          </image>
-          <clip>
-            <near>0.05</near>
-            <far>3</far>
-          </clip>
-        </camera>
-        <plugin name="camera_plugin" filename="libgazebo_ros_openni_kinect.so">
-          <baseline>0.2</baseline>
-          <alwaysOn>true</alwaysOn>
-          <!-- Keep this zero, update_rate in the parent <sensor> tag
-            will control the frame rate. -->
-          <updateRate>0.0</updateRate>
-          <cameraName>camera_ir</cameraName>
-          <imageTopicName>/camera/color/image_raw</imageTopicName>
-          <cameraInfoTopicName>/camera/color/camera_info</cameraInfoTopicName>
-          <depthImageTopicName>/camera/depth/image_raw</depthImageTopicName>
-          <depthImageCameraInfoTopicName>/camera/depth/camera_info</depthImageCameraInfoTopicName>
-          <pointCloudTopicName>/camera/depth/points</pointCloudTopicName>
-          <frameName>depth_camera_link</frameName>
-          <pointCloudCutoff>0.5</pointCloudCutoff>
-          <pointCloudCutoffMax>3.0</pointCloudCutoffMax>
-          <distortionK1>0</distortionK1>
-          <distortionK2>0</distortionK2>
-          <distortionK3>0</distortionK3>
-          <distortionT1>0</distortionT1>
-          <distortionT2>0</distortionT2>
-          <CxPrime>0</CxPrime>
-          <Cx>0</Cx>
-          <Cy>0</Cy>
-          <focalLength>0</focalLength>
-          <hackBaseline>0</hackBaseline>
-        </plugin>
-      </sensor>
-  </gazebo>
+    <gazebo reference = "${prefix}depth_camera_link">
+      <sensor name="camera" type="depth">
+          <update_rate>20</update_rate>
+          <camera>
+            <horizontal_fov>1.047198</horizontal_fov>
+            <image>
+              <width>640</width>
+              <height>480</height>
+              <format>R8G8B8</format>
+            </image>
+            <clip>
+              <near>0.05</near>
+              <far>3</far>
+            </clip>
+          </camera>
+          <plugin name="camera_plugin" filename="libgazebo_ros_openni_kinect.so">
+            <baseline>0.2</baseline>
+            <alwaysOn>true</alwaysOn>
+            <!-- Keep this zero, update_rate in the parent <sensor> tag
+              will control the frame rate. -->
+            <updateRate>0.0</updateRate>
+            <cameraName>camera_ir</cameraName>
+            <imageTopicName>/camera/color/image_raw</imageTopicName>
+            <cameraInfoTopicName>/camera/color/camera_info</cameraInfoTopicName>
+            <depthImageTopicName>/camera/depth/image_raw</depthImageTopicName>
+            <depthImageCameraInfoTopicName>/camera/depth/camera_info</depthImageCameraInfoTopicName>
+            <pointCloudTopicName>/camera/depth/points</pointCloudTopicName>
+            <frameName>depth_camera_link</frameName>
+            <pointCloudCutoff>0.5</pointCloudCutoff>
+            <pointCloudCutoffMax>3.0</pointCloudCutoffMax>
+            <distortionK1>0</distortionK1>
+            <distortionK2>0</distortionK2>
+            <distortionK3>0</distortionK3>
+            <distortionT1>0</distortionT1>
+            <distortionT2>0</distortionT2>
+            <CxPrime>0</CxPrime>
+            <Cx>0</Cx>
+            <Cy>0</Cy>
+            <focalLength>0</focalLength>
+            <hackBaseline>0</hackBaseline>
+          </plugin>
+        </sensor>
+    </gazebo>
     <joint name="${prefix}wrist_3_joint" type="revolute">
       <parent link="${prefix}wrist_2_link" />

Commit message: Added optical camera frame.

File: src/ur_description/urdf/ur10.urdf.xacro (robot description, xacro)
@@ -290,6 +290,20 @@
       <parent link="${prefix}gripper_link" />
       <child link = "${prefix}depth_camera_link" />
-      <origin xyz="0.0 -0.0151 0.0" rpy="0.0 0.0 0.0" />
-    </joint>
+      <origin xyz="0.0 -0.0151 0.0" rpy="0.0 ${-pi/2.0} 0.0" />
+    </joint>
+    <!-- generate an optical frame
+    http://www.ros.org/reps/rep-0103.html#suffix-frames
+    so that ros and opencv can operate on the camera frame correctly
+    -->
+    <joint name="camera_optical_joint" type="fixed">
+      <!-- these values have to be these values otherwise the gazebo camera
+          image won't be aligned properly with the frame it is supposedly
+          originating from -->
+      <origin xyz="0 0 0" rpy="${-pi/2} 0 ${-pi/2}"/>
+      <parent link="depth_camera_link"/>
+      <child link="depth_camera_link_optical"/>
+    </joint>
+    <link name="depth_camera_link_optical">
+    </link>
     <gazebo reference = "${prefix}depth_camera_link">
       <sensor name="camera" type="depth">
@@ -319,5 +333,5 @@
             <depthImageCameraInfoTopicName>/camera/depth/camera_info</depthImageCameraInfoTopicName>
             <pointCloudTopicName>/camera/depth/points</pointCloudTopicName>
-            <frameName>depth_camera_link</frameName>
+            <frameName>depth_camera_link_optical</frameName>
             <pointCloudCutoff>0.5</pointCloudCutoff>
             <pointCloudCutoffMax>3.0</pointCloudCutoffMax>

Commit message: Fixed inertia of camera.

File: src/ur_description/urdf/ur10.urdf.xacro (robot description, xacro)
@@ -35,4 +35,5 @@
     <xacro:property name="wrist_3_mass" value="0.202" />
     <xacro:property name="gripper_mass" value="1.00" />
+    <xacro:property name="camera_mass" value="0.20" />
     <!-- These parameters are borrowed from the urcontrol.conf file
         but are not verified for the correct permutation.
@@ -268,12 +269,7 @@
     </link>
     <link name="${prefix}depth_camera_link">
-    <inertial>
-        <origin xyz="0.0 0.0 0.05" rpy="0 0 0"/>
-        <mass value="1"/>
-        <inertia
-        ixx="1.0" ixy="0.0" ixz="0.0"
-        iyy="1.0" iyz="0.0"
-        izz="1.0"/>
-      </inertial>
+      <xacro:cylinder_inertial radius="0.03" length="0.03" mass="${camera_mass}">
+        <origin xyz="0.1 -0.0151 0.0" rpy="0.0 ${-pi/2.0} 0.0" />
+      </xacro:cylinder_inertial>
       <collision name="collisionBox">
         <geometry>
@@ -290,5 +286,5 @@
       <parent link="${prefix}gripper_link" />
       <child link = "${prefix}depth_camera_link" />
-      <origin xyz="0.0 -0.0151 0.0" rpy="0.0 ${-pi/2.0} 0.0" />
+      <origin xyz="0.1 -0.0151 0.0" rpy="0.0 ${-pi/2.0} 0.0" />
     </joint>
     <!-- generate an optical frame

Commit message: Fixed camera rotation for image data.

File: src/ur_description/urdf/ur10.urdf.xacro (robot description, xacro)
@@ -268,4 +268,77 @@
       </xacro:cylinder_inertial>
     </link>
+    <joint name="${prefix}wrist_3_joint" type="revolute">
+      <parent link="${prefix}wrist_2_link" />
+      <child link = "${prefix}wrist_3_link" />
+      <origin xyz="0.0 0.0 ${wrist_2_length}" rpy="0.0 0.0 0.0" />
+      <axis xyz="0 1 0" />
+      <xacro:unless value="${joint_limited}">
+        <limit lower="${-2.0 * pi}" upper="${2.0 * pi}" effort="54.0" velocity="3.2"/>
+        <xacro:if value="${safety_limits}">
+          <safety_controller soft_lower_limit="${-2.0 * pi + safety_pos_margin}" soft_upper_limit="${2.0 * pi - safety_pos_margin}" k_position="${safety_k_position}" k_velocity="0.0"/>
+        </xacro:if>
+      </xacro:unless>
+      <xacro:if value="${joint_limited}">
+        <limit lower="${wrist_3_lower_limit}" upper="${wrist_3_upper_limit}" effort="54.0" velocity="3.2"/>
+        <xacro:if value="${safety_limits}">
+          <safety_controller soft_lower_limit="${wrist_3_lower_limit + safety_pos_margin}" soft_upper_limit="${wrist_3_upper_limit - safety_pos_margin}" k_position="${safety_k_position}" k_velocity="0.0"/>
+        </xacro:if>
+      </xacro:if>
+      <dynamics damping="0.0" friction="0.0"/>
+    </joint>
+    <link name="${prefix}wrist_3_link">
+      <visual>
+        <geometry>
+          <mesh filename="package://ur_description/meshes/ur10/visual/wrist3.dae"/>
+        </geometry>
+        <material name="LightGrey">
+          <color rgba="0.7 0.7 0.7 1.0"/>
+        </material>
+      </visual>
+      <collision>
+        <geometry>
+          <mesh filename="package://ur_description/meshes/ur10/collision/wrist3.stl"/>
+        </geometry>
+      </collision>
+      <xacro:cylinder_inertial radius="0.045" length="0.0305" mass="${wrist_3_mass}">
+        <origin xyz="0.0 ${wrist_3_length - 0.0305/2} 0.0" rpy="${pi/2} 0 0" />
+      </xacro:cylinder_inertial>
+    </link>
+    <joint name="${prefix}ee_fixed_joint" type="fixed">
+      <parent link="${prefix}wrist_3_link" />
+      <child link = "${prefix}ee_link" />
+      <origin xyz="0.0 ${wrist_3_length} 0.0" rpy="0.0 0.0 ${pi/2.0}" />
+    </joint>
+    <link name="${prefix}ee_link">
+      <collision>
+        <geometry>
+          <box size="0.01 0.01 0.01"/>
+        </geometry>
+        <origin rpy="0 0 0" xyz="-0.01 0 0"/>
+      </collision>
+    </link>
+    <joint name="${prefix}gripper_fixed_joint" type="fixed">
+      <parent link="${prefix}ee_link" />
+      <child link = "${prefix}gripper_link" />
+      <origin xyz="0.0 -0.05 0.1" rpy="0.0 ${pi/2.0} 0.0" />
+    </joint>
+    <link name="${prefix}gripper_link">
+      <visual>
+        <geometry>
+          <mesh filename="package://ur_description/meshes/ur10/visual/gripper.dae"/>
+        </geometry>
+        <material name="LightGrey">
+          <color rgba="0.7 0.7 0.7 1.0"/>
+        </material>
+      </visual>
+      <collision>
+        <geometry>
+          <mesh filename="package://ur_description/meshes/ur10/collision/gripper.stl"/>
+        </geometry>
+      </collision>
+      <xacro:cylinder_inertial radius="0.1" length="0.07" mass="${gripper_mass}">
+        <origin xyz="0.0 -0.05 0.1" rpy="0.0 ${pi/2.0} 0.0" />
+      </xacro:cylinder_inertial>
+    </link>
     <link name="${prefix}depth_camera_link">
       <xacro:cylinder_inertial radius="0.03" length="0.03" mass="${camera_mass}">
@@ -286,5 +359,5 @@
       <parent link="${prefix}gripper_link" />
       <child link = "${prefix}depth_camera_link" />
-      <origin xyz="0.1 -0.0151 0.0" rpy="0.0 ${-pi/2.0} 0.0" />
+      <origin xyz="0.1 -0.0151 0.0" rpy="${pi} ${-pi/2.0} 0.0" />
     </joint>
     <!-- generate an optical frame
@@ -345,77 +418,4 @@
         </sensor>
     </gazebo>
-    <joint name="${prefix}wrist_3_joint" type="revolute">
-      <parent link="${prefix}wrist_2_link" />
-      <child link = "${prefix}wrist_3_link" />
-      <origin xyz="0.0 0.0 ${wrist_2_length}" rpy="0.0 0.0 0.0" />
-      <axis xyz="0 1 0" />
-      <xacro:unless value="${joint_limited}">
-        <limit lower="${-2.0 * pi}" upper="${2.0 * pi}" effort="54.0" velocity="3.2"/>
-        <xacro:if value="${safety_limits}">
-          <safety_controller soft_lower_limit="${-2.0 * pi + safety_pos_margin}" soft_upper_limit="${2.0 * pi - safety_pos_margin}" k_position="${safety_k_position}" k_velocity="0.0"/>
-        </xacro:if>
-      </xacro:unless>
-      <xacro:if value="${joint_limited}">
-        <limit lower="${wrist_3_lower_limit}" upper="${wrist_3_upper_limit}" effort="54.0" velocity="3.2"/>
-        <xacro:if value="${safety_limits}">
-          <safety_controller soft_lower_limit="${wrist_3_lower_limit + safety_pos_margin}" soft_upper_limit="${wrist_3_upper_limit - safety_pos_margin}" k_position="${safety_k_position}" k_velocity="0.0"/>
-        </xacro:if>
-      </xacro:if>
-      <dynamics damping="0.0" friction="0.0"/>
-    </joint>
-    <link name="${prefix}wrist_3_link">
-      <visual>
-        <geometry>
-          <mesh filename="package://ur_description/meshes/ur10/visual/wrist3.dae"/>
-        </geometry>
-        <material name="LightGrey">
-          <color rgba="0.7 0.7 0.7 1.0"/>
-        </material>
-      </visual>
-      <collision>
-        <geometry>
-          <mesh filename="package://ur_description/meshes/ur10/collision/wrist3.stl"/>
-        </geometry>
-      </collision>
-      <xacro:cylinder_inertial radius="0.045" length="0.0305" mass="${wrist_3_mass}">
-        <origin xyz="0.0 ${wrist_3_length - 0.0305/2} 0.0" rpy="${pi/2} 0 0" />
-      </xacro:cylinder_inertial>
-    </link>
-    <joint name="${prefix}ee_fixed_joint" type="fixed">
-      <parent link="${prefix}wrist_3_link" />
-      <child link = "${prefix}ee_link" />
-      <origin xyz="0.0 ${wrist_3_length} 0.0" rpy="0.0 0.0 ${pi/2.0}" />
-    </joint>
-    <link name="${prefix}ee_link">
-      <collision>
-        <geometry>
-          <box size="0.01 0.01 0.01"/>
-        </geometry>
-        <origin rpy="0 0 0" xyz="-0.01 0 0"/>
-      </collision>
-    </link>
-    <joint name="${prefix}gripper_fixed_joint" type="fixed">
-      <parent link="${prefix}ee_link" />
-      <child link = "${prefix}gripper_link" />
-      <origin xyz="0.0 -0.05 0.1" rpy="0.0 ${pi/2.0} 0.0" />
-    </joint>
-    <link name="${prefix}gripper_link">
-      <visual>
-        <geometry>
-          <mesh filename="package://ur_description/meshes/ur10/visual/gripper.dae"/>
-        </geometry>
-        <material name="LightGrey">
-          <color rgba="0.7 0.7 0.7 1.0"/>
-        </material>
-      </visual>
-      <collision>
-        <geometry>
-          <mesh filename="package://ur_description/meshes/ur10/collision/gripper.stl"/>
-        </geometry>
-      </collision>
-      <xacro:cylinder_inertial radius="0.1" length="0.07" mass="${gripper_mass}">
-        <origin xyz="0.0 -0.05 0.1" rpy="0.0 ${pi/2.0} 0.0" />
-      </xacro:cylinder_inertial>
-    </link>
     <xacro:ur_arm_transmission prefix="${prefix}" hw_interface="${transmission_hw_interface}" />
     <xacro:ur_arm_gazebo prefix="${prefix}" />

Commit message: Fixed image rotation of camera.

File: src/ur_description/urdf/ur10.urdf.xacro (robot description, xacro)
@@ -359,5 +359,5 @@
       <parent link="${prefix}gripper_link" />
       <child link = "${prefix}depth_camera_link" />
-      <origin xyz="0.1 -0.0151 0.0" rpy="${pi} ${-pi/2.0} 0.0" />
+      <origin xyz="0.1 -0.0151 0.0" rpy="${pi/2.0} ${-pi/2.0} 0.0" />
     </joint>
     <!-- generate an optical frame
